File: board/smoke_gira/Gira.kicad_pcb (KiCad board)
At the start: 2 copper layers, 38 x 65 mm, 13 parts, among them J1 Moat_Bus_wire, J2 1wireConn, J3 I2C

Commit message: Too many reworks to count.
Most notably: Split GND and GNDPWR.
Parts:
- removed the REF** at (154.5, 108.0)
- added J4: Conn_01x06, Connector_PinSocket_2.54mm:PinSocket_1x06_P2.54mm_Vertical, F.Cu at (151.8, 104.6)
- added REF**: OSHW-Logo_5.7x6mm_Copper, Symbol:OSHW-Logo_5.7x6mm_Copper, F.Cu at (132.9, 79.9)
Connections:
- J1 pad 10: (no net) -> +12V
- J1 pad 23: GND -> GNDPWR
- J1 pad 24: GND -> GNDPWR
- J1 pad 3: (no net) -> Net-(J1-Pad3)
- J1 pad 4: (no net) -> Net-(J1-Pad4)
- J1 pad 6: (no net) -> Net-(J1-Pad6)
- J1 pad 8: (no net) -> Net-(J1-Pad8)
Routing:
- net Net-(J1-Pad6): track 0.00 -> 42.7 mm, vias 0 -> 1
- net Net-(J1-Pad8): track 0.00 -> 37.4 mm, vias 0 -> 1
- net Net-(J1-Pad3): track 0.00 -> 33.8 mm, vias 0 -> 3
- net +3V3: track 63.3 -> 95.4 mm, vias 4 -> 5
- net Net-(J1-Pad4): track 0.00 -> 31.5 mm, vias 0 -> 1
- net GND: track 121.1 -> 138.1 mm, vias 9 -> 10
- net /SCL: track 39.2 -> 52.5 mm
- net +5V: track 53.7 -> 66.8 mm, vias 1 -> 2
- net +12V: track 51.9 -> 63.7 mm
- net /SDA: track 42.8 -> 50.3 mm
- net GNDPWR: track 0.00 -> 6.19 mm, vias 0 -> 1
- net /Unk_2: track 53.3 -> 59.5 mm
- net /1wire: track 47.0 -> 51.5 mm
- net Net-(Bus3-Pad1): track 48.1 -> 52.1 mm
- net Net-(Bus2-Pad1): track 31.5 -> 33.2 mm
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Other:
- board size 38 x 65 mm -> 38 x 53.2 mm
- board text added: "1"
- board text added: "2"
- board text added: "R"
- board text added: "T"
- board text added: "v2.5"
- board text removed: "v2.3"
