File: wire_16/plug16.kicad_pcb (KiCad board)
At the start: 2 copper layers, 18.8 x 20.4 mm, 2 parts, among them J1 Moat_Wire_16, J2 Moat_Wire_12

Commit message: wixup wire_16
Routing:
- net /GND: vias 19 -> 18
Other:
- board text added: "MoaT Wire 16"
- board text added: "V 2.0"
- board text removed: "MoaT wire 16"
Changed lines of the file:
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@@
   (gr_line (start 38 44.7) (end 38 57.7) (layer "Edge.Cuts") (width 0.15))
   (gr_line (start 19.2 61.9) (end 19.2 41.45) (layer "Edge.Cuts") (width 0.15))
-  (gr_text "MoaT\nwire 16" (at 35.78 51.348 90) (layer "F.SilkS")
+  (gr_text "V 2.0" (at 32.7 54.7) (layer "F.SilkS")
+    (effects (font (size 1 1) (thickness 0.2)))
+  )
+  (gr_text "MoaT\nWire 16" (at 35.78 51.348 90) (layer "F.SilkS")
     (effects (font (size 1 1) (thickness 0.2)))
   )
@@
   (segment (start 30.804511 47.050489) (end 32.399511 47.050489) (width 0.5) (layer "B.Cu") (net 2))
   (segment (start 32.399511 47.050489) (end 32.527375 46.922625) (width 0.5) (layer "B.Cu") (net 2))
+  (segment (start 21.55 43.7) (end 27.15 43.7) (width 0.5) (layer "B.Cu") (net 2))
   (segment (start 30.73 47.125) (end 30.804511 47.050489) (width 0.5) (layer "B.Cu") (net 2))
-  (segment (start 30.309956 42.95) (end 31.25 43.890044) (width 0.5) (layer "B.Cu") (net 2))
-  (segment (start 27.9 42.95) (end 27.15 43.7) (width 0.5) (layer "B.Cu") (net 2))
   (segment (start 31.25 43.890044) (end 31.25 44.415498) (width 0.5) (layer "B.Cu") (net 2))
-  (segment (start 21.55 43.7) (end 20.8 42.95) (width 0.5) (layer "B.Cu") (net 2))
-  (segment (start 27.15 43.7) (end 21.55 43.7) (width 0.5) (layer "B.Cu") (net 2))
-  (segment (start 27.9 42.95) (end 30.309956 42.95) (width 0.5) (layer "B.Cu") (net 2))
+  (segment (start 20.8 42.95) (end 21.55 43.7) (width 0.5) (layer "B.Cu") (net 2))
+  (segment (start 27.649511 43.200489) (end 30.560445 43.200489) (width 0.5) (layer "B.Cu") (net 2))
+  (segment (start 27.15 43.7) (end 27.649511 43.200489) (width 0.5) (layer "B.Cu") (net 2))
+  (segment (start 30.560445 43.200489) (end 31.25 43.890044) (width 0.5) (layer "B.Cu") (net 2))
+  (segment (start 34.5 44.6) (end 35.5 45.6) (width 0.5) (layer "F.Cu") (net 3))
+  (segment (start 31.5 43.45) (end 32.65 44.6) (width 0.5) (layer "F.Cu") (net 3))
+  (segment (start 30.75 43.45) (end 31.5 43.45) (width 0.5) (layer "F.Cu") (net 3))
+  (segment (start 35.5 45.6) (end 35.5 46.95) (width 0.5) (layer "F.Cu") (net 3))
+  (segment (start 32.65 44.6) (end 34.5 44.6) (width 0.5) (layer "F.Cu") (net 3))
   (segment (start 30.25 43.95) (end 30.75 43.45) (width 0.5) (layer "F.Cu") (net 3))
-  (segment (start 31.5 43.45) (end 32.5 44.45) (width 0.5) (layer "F.Cu") (net 3))
-  (segment (start 30.75 43.45) (end 31.5 43.45) (width 0.5) (layer "F.Cu") (net 3))
-  (segment (start 35.5 45.45) (end 35.5 46.95) (width 0.5) (layer "F.Cu") (net 3))
-  (segment (start 32.5 44.45) (end 34.5 44.45) (width 0.5) (layer "F.Cu") (net 3))
-  (segment (start 34.5 44.45) (end 35.5 45.45) (width 0.5) (layer "F.Cu") (net 3))
   (via (at 30.25 43.95) (size 0.7) (drill 0.4) (layers "F.Cu" "B.Cu") (net 3))
   (via (at 35.5 46.95) (size 0.7) (drill 0.4) (layers "F.Cu" "B.Cu") (net 3))
@@
   (via (at 24.5 59.7) (size 0.7) (drill 0.4) (layers "F.Cu" "B.Cu") (free) (net 4))
   (via (at 35.5 58.2) (size 0.7) (drill 0.4) (layers "F.Cu" "B.Cu") (free) (net 4))
-  (via (at 31.20312 42.7005) (size 0.7) (drill 0.4) (layers "F.Cu" "B.Cu") (free) (net 4))
-  (via (at 32.75 43.45) (size 0.7) (drill 0.4) (layers "F.Cu" "B.Cu") (free) (net 4))
+  (via (at 33.1 43.7) (size 0.7) (drill 0.4) (layers "F.Cu" "B.Cu") (free) (net 4))
   (via (at 34.5 47.45) (size 0.7) (drill 0.4) (layers "F.Cu" "B.Cu") (free) (net 4))
   (via (at 30 59.7) (size 0.7) (drill 0.4) (layers "F.Cu" "B.Cu") (free) (net 4))
