File: old/board/heating12/plug16.kicad_pcb (KiCad board)
At the start: 2 copper layers, 40.7 x 47.4 mm, 17 parts, among them J1 Moat_Bus_16, J10 1wireConn, J2 Moat_Bus_wire, J3 SCLK, J4 SDA, J5 3V3, J6 GND, J7 Conn_01x05, J8 S1, J9 S2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

Commit message: format update
Other:
- net class Default removed
- net class Power removed
