File: old/misc/PiPower/PiPower.kicad_pcb (KiCad board)
At the start: 2 copper layers, 56 x 65 mm, 128 parts, among them J1 Raspberry_Pi_2_3, J10 Out 6, J2 Power, J3 Out 0, J4 Out 1, J5 Out 2, J6 Out 3, J7 Out 4, J8 Out 5, J9 Out 7, U1 MP5014A, U10 INA219AxD, U11 MP5014A, U12 MP5014A, U13 MP5014A, U14 INA219AxD, U15 INA219AxD, U16 INA219AxD, U17 PCAL6416APW, U2 INA219AxD, U3 MP5014A, U4 MP5014A, U5 MP5014A, U6 INA219AxD, U7 INA219AxD, U8 MP5014A, U9 INA219AxD

Commit message: PiPower: kicad 6.99 update
Parts:
- R13: renamed from R9; footprint Resistor_SMD:R_0805_2012Metric_Pad1.20x1.40mm_HandSolder -> Resistor_SMD:R_0805_2012Metric
- R19: renamed from R41; footprint Resistor_SMD:R_0603_1608Metric_Pad0.98x0.95mm_HandSolder -> Resistor_SMD:R_0603_1608Metric
- R23: renamed from R12; footprint Resistor_SMD:R_0805_2012Metric_Pad1.20x1.40mm_HandSolder -> Resistor_SMD:R_0805_2012Metric
- R29: renamed from R40; footprint Resistor_SMD:R_0603_1608Metric_Pad0.98x0.95mm_HandSolder -> Resistor_SMD:R_0603_1608Metric
- R3: footprint Resistor_SMD:R_0805_2012Metric_Pad1.20x1.40mm_HandSolder -> Resistor_SMD:R_0805_2012Metric
- R33: renamed from R15; footprint Resistor_SMD:R_0805_2012Metric_Pad1.20x1.40mm_HandSolder -> Resistor_SMD:R_0805_2012Metric
- R39: footprint Resistor_SMD:R_0603_1608Metric_Pad0.98x0.95mm_HandSolder -> Resistor_SMD:R_0603_1608Metric
- R43: renamed from R19; footprint Resistor_SMD:R_0805_2012Metric_Pad1.20x1.40mm_HandSolder -> Resistor_SMD:R_0805_2012Metric
- R49: renamed from R38; footprint Resistor_SMD:R_0603_1608Metric_Pad0.98x0.95mm_HandSolder -> Resistor_SMD:R_0603_1608Metric
- R53: renamed from R26; footprint Resistor_SMD:R_0805_2012Metric_Pad1.20x1.40mm_HandSolder -> Resistor_SMD:R_0805_2012Metric
- R59: renamed from R37; footprint Resistor_SMD:R_0603_1608Metric_Pad0.98x0.95mm_HandSolder -> Resistor_SMD:R_0603_1608Metric
- R63: renamed from R31; footprint Resistor_SMD:R_0805_2012Metric_Pad1.20x1.40mm_HandSolder -> Resistor_SMD:R_0805_2012Metric
- R69: renamed from R36; footprint Resistor_SMD:R_0603_1608Metric_Pad0.98x0.95mm_HandSolder -> Resistor_SMD:R_0603_1608Metric
- R7: renamed from R33; footprint Resistor_SMD:R_0603_1608Metric_Pad0.98x0.95mm_HandSolder -> Resistor_SMD:R_0603_1608Metric
- R73: renamed from R27; footprint Resistor_SMD:R_0805_2012Metric_Pad1.20x1.40mm_HandSolder -> Resistor_SMD:R_0805_2012Metric
- R79: renamed from R35; footprint Resistor_SMD:R_0603_1608Metric_Pad0.98x0.95mm_HandSolder -> Resistor_SMD:R_0603_1608Metric
- R8: renamed from R34; footprint Resistor_SMD:R_0603_1608Metric_Pad0.98x0.95mm_HandSolder -> Resistor_SMD:R_0603_1608Metric
- R9: renamed from R42; footprint Resistor_SMD:R_0603_1608Metric_Pad0.98x0.95mm_HandSolder -> Resistor_SMD:R_0603_1608Metric
- renumbered R5 to R11, R8 to R12, R11 to R14, R6 to R21, R10 to R22, R14 to R24, R7 to R31, R13 to R32, R16 to R34, R17 to R41, R18 to R42, R20 to R44, R21 to R51, R24 to R52, R28 to R54, R23 to R61, R30 to R62, R32 to R64, R22 to R71, R25 to R72, R29 to R74
Connections:
- J1 pad 10: (no net) -> unconnected-(J1-GPIO15/RXD)
- J1 pad 11: (no net) -> unconnected-(J1-GPIO17)
- J1 pad 12: (no net) -> unconnected-(J1-GPIO18/PWM0)
- J1 pad 13: (no net) -> unconnected-(J1-GPIO27)
- J1 pad 14: (no net) -> unconnected-(J1-GND)_1
- J1 pad 15: (no net) -> unconnected-(J1-GPIO22)
- J1 pad 16: (no net) -> unconnected-(J1-GPIO23)
- J1 pad 17: (no net) -> unconnected-(J1-3V3)
- J1 pad 18: (no net) -> unconnected-(J1-GPIO24)
- J1 pad 19: (no net) -> unconnected-(J1-MOSI0/GPIO10)
- J1 pad 2: (no net) -> unconnected-(J1-5V)_1
- J1 pad 20: (no net) -> unconnected-(J1-GND)_2
- J1 pad 21: (no net) -> unconnected-(J1-MISO0/GPIO9)
- J1 pad 22: (no net) -> unconnected-(J1-GPIO25)
- J1 pad 23: (no net) -> unconnected-(J1-SCLK0/GPIO11)
- J1 pad 24: (no net) -> unconnected-(J1-~{CE0}/GPIO8)
- J1 pad 25: (no net) -> unconnected-(J1-GND)_3
- J1 pad 26: (no net) -> unconnected-(J1-~{CE1}/GPIO7)
- J1 pad 27: (no net) -> unconnected-(J1-ID_SD/GPIO0)
- J1 pad 28: (no net) -> unconnected-(J1-ID_SC/GPIO1)
- J1 pad 29: (no net) -> unconnected-(J1-GCLK1/GPIO5)
- J1 pad 30: (no net) -> unconnected-(J1-GND)_4
- J1 pad 31: (no net) -> unconnected-(J1-GCLK2/GPIO6)
- J1 pad 32: (no net) -> unconnected-(J1-PWM0/GPIO12)
- J1 pad 33: (no net) -> unconnected-(J1-PWM1/GPIO13)
- J1 pad 34: (no net) -> unconnected-(J1-GND)_5
- J1 pad 35: (no net) -> unconnected-(J1-GPIO19/MISO1)
- J1 pad 36: (no net) -> unconnected-(J1-GPIO16)
- J1 pad 37: (no net) -> unconnected-(J1-GPIO26)
- J1 pad 38: (no net) -> unconnected-(J1-GPIO20/MOSI1)
- J1 pad 39: (no net) -> unconnected-(J1-GND)_6
- J1 pad 4: (no net) -> unconnected-(J1-5V)
- J1 pad 40: (no net) -> unconnected-(J1-GPIO21/SCLK1)
- J1 pad 8: (no net) -> unconnected-(J1-GPIO14/TXD)
- J1 pad 9: (no net) -> unconnected-(J1-GND)
Routing:
- net +3V3: track 427.4 -> 418.5 mm
- net SDA: track 335.7 -> 336.8 mm
- net SCL: track 360.5 -> 360.0 mm
Other:
- board text added: "JLCJLCJLCJLC"
