File: old/misc/PiPower/PiPower.kicad_sch (KiCad schematic)
At the start: 34 parts, among them J1 Raspberry_Pi_2_3, J2 Power, J3 Out 0, U1 MP5014A, U17 PCAL6416APW, U2 INA219AxD

Commit message: PiPower: kicad 6.99 update
Parts:
- C1, C3: symbol localstuff:CP -> localparts:CP_10µ_16V_0603; LCSC (none) -> C70225
- C2, J3: now left out of the parts list
- C4, C41: symbol localstuff:CP -> localparts:CP_100n_50V_0603; LCSC (none) -> C14663
- C5: symbol Device:C -> localparts:CP_1µ_50V_0603; LCSC (none) -> C15849
- R1: symbol localstuff:R -> localparts:R_22_0603; JLC (none) -> C23345; LCSC (none) -> C23345
- R19, R29, R39, R49, R59, R69, R79, R9: footprint Resistor_SMD:R_0603_1608Metric_Pad0.98x0.95mm_HandSolder -> Resistor_SMD:R_0603_1608Metric; symbol localstuff:R -> localparts:R_10k_0603; LCSC (none) -> C25804
- R2: symbol localstuff:R -> localparts:R_10_0603; JLC (none) -> C22859; LCSC (none) -> C22859
- R3: footprint Resistor_SMD:R_0805_2012Metric_Pad1.20x1.40mm_HandSolder -> Resistor_SMD:R_0805_2012Metric; symbol localstuff:R -> localparts:R_X1_0805; JLC (none) -> C23345; LCSC (none) -> C23345
- R4: symbol localstuff:R -> localparts:R_10_0603; LCSC (none) -> C22859
- R7, R8: footprint Resistor_SMD:R_0603_1608Metric_Pad0.98x0.95mm_HandSolder -> Resistor_SMD:R_0603_1608Metric; symbol localstuff:R -> localparts:R_1k_0603; LCSC (none) -> C328340
- U2: symbol Analog_ADC:INA219AxD -> localstuff:INA219AxD; LCSC (none) -> C138706
