File: old/misc/PiPower/seven.kicad_sch (KiCad schematic)
At the start: 84 parts, among them J10 Out 6, J4 Out 1, J5 Out 2, J6 Out 3, J7 Out 4, J8 Out 5, J9 Out 7, U10 INA219AxD, U11 MP5014A, U12 MP5014A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

Commit message: PiPower: kicad 6.99 update
Parts:
- C10, C11, C18, C28, C29, C31, C8, J10, J4, J5, J6, J7, J8, J9: now left out of the parts list
- C12, C13, C15, C17, C23, C26, C27, C30, C32, C33, C36, C6, C7, C9: symbol localstuff:CP -> localparts:CP_10µ_16V_0603; LCSC (none) -> C70225
- C14, C16, C19, C24, C34, C35, C37: symbol localstuff:CP -> localparts:CP_100n_50V_0603; LCSC (none) -> C14663
- C20, C21, C22, C25, C38, C39, C40: symbol Device:C -> localparts:CP_1µ_50V_0603; LCSC (none) -> C15849
- R11, R21, R31, R41, R51, R61, R71: symbol localstuff:R -> localparts:R_22_0603; JLC (none) -> C23345; LCSC (none) -> C23345
- R12, R14, R22, R24, R32, R34, R42, R44, R52, R54, R62, R64, R72, R74: symbol localstuff:R -> localparts:R_10_0603; LCSC (none) -> C22859
- R13, R23, R33, R43, R53, R63, R73: footprint Resistor_SMD:R_0805_2012Metric_Pad1.20x1.40mm_HandSolder -> Resistor_SMD:R_0805_2012Metric; symbol localstuff:R -> localparts:R_X1_0805; JLC (none) -> C23345; LCSC (none) -> C23345
- U10, U14, U15, U16, U6, U7, U9: symbol Analog_ADC:INA219AxD -> localstuff:INA219AxD; LCSC (none) -> C138706
