File: base/gira/base_gira.kicad_pcb (KiCad board)
At the start: 2 copper layers, 38 x 53.2 mm, 19 parts, among them J1 Moat_Bus_wire, J2 1wireConn, J3 I2C, J4 Conn_01x06, Q1 2N7002

Commit message: Finish rename
Routing:
- net GND: track 131.5 -> 133.4 mm, vias 11 -> 19
- net /1wire_5: track 7.21 -> 9.00 mm
