File: bms/HXS/HXS.kicad_pcb (KiCad board)
At the start: 2 copper layers, 33.4 x 19.5 mm, 10 parts, among them J1 Power, J2 Conn_LEM_5, U1 HXS50-NP

Commit message: BMS stuff update
Parts:
- moved C1 6.60 mm to (65.9, 46.2), turned to -90 degrees
- moved C2 6.60 mm to (65.9, 52.8), turned to -90 degrees
- moved J2 5.98 mm to (61.5, 52.4), turned to 90 degrees
- moved U1 0.41 mm to (75.8, 49.4)
- turned C3 to -90 degrees
Connections:
- J1 pad 1: Net-(J1-Pin_1) -> Net-(U1-Pad8)
- U1 pad 1: Net-(J1-Pin_1) -> Net-(J1-Pin_2)
- U1 pad 8: Net-(J1-Pin_2) -> Net-(U1-Pad8)
Routing:
- net Net-(U1-Pad8): track 0.00 -> 15.2 mm
- net Net-(J1-Pin_2): track 15.5 -> 7.14 mm
- net Net-(J1-Pin_1): track 7.54 -> 0.00 mm
- net Net-(J2-GND): track 22.6 -> 21.5 mm
- net Net-(J2-+): track 17.8 -> 16.9 mm
- net Net-(J2-Out): track 9.35 -> 8.59 mm
- net Net-(J2-Ref): track 9.90 -> 9.18 mm
