File: bms/HXS/HXS.kicad_sch (KiCad schematic)
At the start: 6 parts, among them J1 Power, J2 Conn_LEM_5, U1 HXS50-NP

Commit message: BMS stuff update
Connections:
- net at U1.1: now also J1.2 (Pin_2); no longer J1.1 (Pin_1)
- net at U1.8: now also J1.1 (Pin_1); no longer J1.2 (Pin_2)
Other:
- moved on the sheet: J1
Changed lines of the file:
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@@
     (stroke (width 0) (type default))
   )
-  (wire (pts (xy 66.04 55.88) (xy 68.58 55.88))
+  (wire (pts (xy 62.23 55.88) (xy 68.58 55.88))
     (stroke (width 0) (type default))
   )
@@
     (stroke (width 0) (type default))
   )
-  (wire (pts (xy 66.04 63.5) (xy 66.04 68.58))
+  (wire (pts (xy 66.04 58.42) (xy 66.04 68.58))
     (stroke (width 0) (type default))
   )
   (wire (pts (xy 93.98 52.07) (xy 93.98 68.58))
-    (stroke (width 0) (type default))
-  )
-  (wire (pts (xy 63.5 60.96) (xy 66.04 60.96))
     (stroke (width 0) (type default))
   )
@@
     (stroke (width 0) (type default))
   )
-  (wire (pts (xy 63.5 63.5) (xy 66.04 63.5))
-    (stroke (width 0) (type default))
-  )
-  (wire (pts (xy 66.04 60.96) (xy 66.04 55.88))
+  (wire (pts (xy 62.23 58.42) (xy 66.04 58.42))
     (stroke (width 0) (type default))
   )
@@
     (pin "2")
   )
-  (symbol (lib_id "Connector:Conn_01x02_Female") (at 58.42 60.96 0) (mirror y) (unit 1)
+  (symbol (lib_id "Connector:Conn_01x02_Female") (at 57.15 58.42 180) (unit 1)
     (in_bom yes) (on_board yes)
-    (property "Reference" "J1" (id 0) (at 58.42 59.69 0)
+    (property "Reference" "J1" (id 0) (at 57.15 59.69 0)
       (effects (font (size 1.27 1.27)))
     )
-    (property "Value" "Power" (id 1) (at 58.42 64.77 0)
+    (property "Value" "Power" (id 1) (at 57.15 54.61 0)
       (effects (font (size 1.27 1.27)))
     )
-    (property "Footprint" "localstuff:Conn_P5.0mm_2_Lumberg" (id 2) (at 58.42 60.96 0)
+    (property "Footprint" "localstuff:Conn_P5.0mm_2_Lumberg" (id 2) (at 57.15 58.42 0)
       (effects (font (size 1.27 1.27)) hide)
     )
-    (property "Datasheet" "~" (id 3) (at 58.42 60.96 0)
+    (property "Datasheet" "~" (id 3) (at 57.15 58.42 0)
       (effects (font (size 1.27 1.27)) hide)
     )
