File: adapt/prog-wire/prog-wire.kicad_pcb (KiCad board)
At the start: 2 copper layers, 9 x 12 mm, 2 parts, among them J1 Conn_01x06

Commit message: misc updates I didn't bother checking in, oops
Parts:
- Prog1: moved to B.Cu
- moved Prog1 0.13 mm to (32.0, 30.9)
Routing:
- net /GND: track 17.8 -> 7.99 mm
- net /RST: track 14.9 -> 6.94 mm
- net /Rx: track 6.81 -> 13.8 mm
- net /Boot0: track 7.03 -> 12.3 mm, vias 0 -> 1
- net /3V3: track 9.95 -> 6.34 mm
- net /Tx: track 7.03 -> 9.71 mm, vias 0 -> 1
Other:
- outline, holes or cut-outs redrawn
