File: base/heating/base_heating.kicad_sch (KiCad schematic)
At the start: 20 parts, among them J1 Moat_Bus_12, J10 1wireConn, J2 Moat_Bus_wire, J3 SCLK, J4 SDA, J5 3V3, J6 GND, J7 Conn_01x05, J8 S1, J9 S2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

Commit message: misc updates I didn't bother checking in, oops
Parts:
- removed J7: Conn_01x05, Connector_PinHeader_2.00mm:PinHeader_1x05_P2.00mm_Vertical, symbol Connector_Generic:Conn_01x05
- added J11: T2, localstuff:1X02_GN, symbol Connector:Conn_01x02_Female
- added J12: T3, localstuff:1X02_GN, symbol Connector:Conn_01x02_Female
- added J7: T1, localstuff:1X02_GN, symbol Connector:Conn_01x02_Female
- added Q4: 2N7002, Package_TO_SOT_SMD:SOT-23, symbol localstuff:2N7002
- added R3: R_1M_0603, Resistor_SMD:R_0603_1608Metric, symbol localparts:R_1M_0603
- added R4, R8, R9: 10k, Resistor_SMD:R_0603_1608Metric, symbol localparts:R_10k_0603
Connections:
- net +3V3: now also J11.1 (Pin_1), J12.1 (Pin_1), J7.1 (Pin_1)
- net GND: now also Q4.2 (S), R3.2
- net T1: now also J7.2 (Pin_2), R4.1
- net T2: now also J11.2 (Pin_2), R8.1
- net T3: now also J12.2 (Pin_2), R9.1
- net ena: now reaches J2.13 (S5)
- net ena: now also Q4.1 (G), R3.1
- new net: Q4.3 (D), R4.2, R8.2, R9.2
- no-connect marks 10 -> 9
