File: base/heating/base_heating.kicad_sch (KiCad schematic)
At the start: 27 parts, among them J1 Moat_Bus_12, J10 1wireConn, J11 T2, J12 T3, J2 Moat_Bus_wire, J3 SCLK, J4 SDA, J5 3V3, J6 GND, J7 T1, J8 S1, J9 S2, Q1 2N7002, Q2 2N7002, Q3 2N7002, Q4 2N7002

Commit message: A host of un-logged changes
Parts:
- added R10, R11: R_1M_0603, Resistor_SMD:R_0603_1608Metric, symbol localparts:R_1M_0603
Connections:
- net GNDPWR: now also R10.2, R11.2
- net S1: now also R10.1
- net S2: now also R11.1
