File: proc/stm32/proc_stm32.kicad_pcb (KiCad board)
At the start: 2 copper layers, 28 x 18.8 mm, 22 parts, among them J1 Moat_Compute_24, Q1 2N7002, Q2 2N7002, Q3 2N7002, Q4 2N7002, U1 MIC5504, U2 STM32L051K8Tx, U3 LTC4311, U4 LTC4311

Commit message: misc updates I didn't bother checking in, oops
Parts:
- removed C6: 100nF, Capacitor_SMD:C_0603_1608Metric
- removed U3, U4: LTC4311, Package_DFN_QFN:ST_UQFN-6L_1.5x1.7mm_Pitch0.5mm
- C1, C2: footprint Capacitor_SMD:C_0603_1608Metric_Pad1.05x0.95mm_HandSolder -> Capacitor_SMD:C_0603_1608Metric
- C3: footprint Capacitor_SMD:C_1206_3216Metric_Pad1.42x1.75mm_HandSolder -> Capacitor_SMD:C_0603_1608Metric
- C4, C5: footprint Capacitor_SMD:C_0603_1608Metric -> Resistor_SMD:R_0603_1608Metric_Pad0.98x0.95mm_HandSolder
- moved R1 6.29 mm to (60.0, 58.2), turned to -135 degrees
- moved C4 5.42 mm to (47.6, 59.3), turned to 180 degrees
- moved Prog1 4.53 mm to (60.8, 56.1), turned to -90 degrees
- moved U1 3.25 mm to (51.0, 58.0), turned to 90 degrees
- moved C5 2.16 mm to (53.9, 58.5), turned to -90 degrees
- moved C2 0.83 mm to (57.1, 58.6)
Routing:
- net +3V3: track 81.4 -> 55.1 mm, vias 6 -> 3
- net /ena: track 44.8 -> 27.8 mm, vias 6 -> 2
- net /Bus1: track 40.3 -> 26.3 mm, vias 7 -> 3
- net /Bus2: track 29.7 -> 17.3 mm, vias 4 -> 2
- net /Bus3: track 30.1 -> 18.7 mm, vias 5 -> 4
- net GND: track 98.2 -> 87.4 mm, vias 5 -> 7
- net /Tx: track 33.4 -> 25.1 mm, vias 4 -> 2
- net +5V: track 36.8 -> 31.5 mm
- net /Bus4: track 35.5 -> 31.1 mm, vias 6 -> 5
- net /Rx: track 36.1 -> 31.9 mm, vias 4 -> 3
- net /Boot0: track 9.28 -> 5.35 mm
- net /1wire: track 21.0 -> 19.4 mm
- net /Bus1_out: track 18.8 -> 20.1 mm
- net /EN: track 8.09 -> 7.19 mm
- net /Bus2_out: track 17.0 -> 17.9 mm
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Other:
- board size 28 x 18.8 mm -> 28 x 15.5 mm
- board text added: "V 3.3"
- board text removed: "V 2.3"
