File: proc/stm32/proc_stm32.kicad_sch (KiCad schematic)
At the start: 21 parts, among them J1 Moat_Compute_24, Q1 2N7002, Q2 2N7002, Q3 2N7002, Q4 2N7002, U1 MIC5504, U2 STM32L051K8Tx, U3 LTC4311, U4 LTC4311

Commit message: misc updates I didn't bother checking in, oops
Parts:
- C1, C2: footprint Capacitor_SMD:C_0603_1608Metric_Pad1.05x0.95mm_HandSolder -> Capacitor_SMD:C_0603_1608Metric; symbol localstuff:C -> localparts:CP_100n_50V_0603; LCSC (none) -> C14663
- C3: footprint Capacitor_SMD:C_1206_3216Metric_Pad1.42x1.75mm_HandSolder -> Capacitor_SMD:C_0603_1608Metric; symbol localstuff:CP -> localparts:CP_10µ_16V_0603; LCSC (none) -> C70225
- C4, C5: footprint Capacitor_SMD:C_0603_1608Metric -> Resistor_SMD:R_0603_1608Metric_Pad0.98x0.95mm_HandSolder; symbol localstuff:CP -> localparts:CP_1µ_50V_0603; LCSC (none) -> C15849
- C6: symbol localstuff:CP -> localparts:CP_100n_50V_0603; LCSC (none) -> C14663; now left out of the parts list
- U2: symbol MCU_ST_STM32L0:STM32L051K8Tx -> localparts:STM32L051K8Tx
- U3, U4: now left out of the parts list
Changed lines of the file:
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@@
     (effects (font (size 1.27 1.27)) (justify right bottom))
   )
-  (symbol (lib_id "localstuff:C") (at 135.89 36.83 0) (unit 1)
+  (symbol (lib_id "localparts:CP_100n_50V_0603") (at 135.89 36.83 0) (unit 1)
     (in_bom yes) (on_board yes)
     (property "Reference" "C2" (id 0) (at 136.525 34.29 0)
@@
       (effects (font (size 1.27 1.27)) (justify left))
     )
-    (property "Footprint" "Capacitor_SMD:C_0603_1608Metric_Pad1.05x0.95mm_HandSolder" (id 2) (at 136.8552 40.64 0)
+    (property "Footprint" "Capacitor_SMD:C_0603_1608Metric" (id 2) (at 136.8552 40.64 0)
       (effects (font (size 1.27 1.27)) hide)
     )
     (property "Datasheet" "" (id 3) (at 135.89 36.83 0)
       (effects (font (size 1.27 1.27)) hide)
+    )
+    (property "LCSC" "C14663" (id 4) (at 135.89 36.83 0)
+      (effects (font (size 1.27 1.27)))
     )
     (pin "1")
@@
     (pin "1")
   )
-  (symbol (lib_id "MCU_ST_STM32L0:STM32L051K8Tx") (at 181.61 120.65 0) (unit 1)
+  (symbol (lib_id "localparts:STM32L051K8Tx") (at 181.61 120.65 0) (unit 1)
     (in_bom yes) (on_board yes)
     (property "Reference" "U2" (id 0) (at 180.34 148.3106 0)
@@
     (pin "1")
   )
-  (symbol (lib_id "localstuff:CP") (at 146.05 36.83 0) (unit 1)
+  (symbol (lib_id "localparts:CP_10µ_16V_0603") (at 146.05 36.83 0) (unit 1)
     (in_bom yes) (on_board yes)
     (property "Reference" "C3" (id 0) (at 146.685 34.29 0)
@@
       (effects (font (size 1.27 1.27)) (justify left))
     )
-    (property "Footprint" "Capacitor_SMD:C_1206_3216Metric_Pad1.42x1.75mm_HandSolder" (id 2) (at 147.0152 40.64 0)
+    (property "Footprint" "Capacitor_SMD:C_0603_1608Metric" (id 2) (at 147.0152 40.64 0)
       (effects (font (size 1.27 1.27)) hide)
     )
@@
       (effects (font (size 1.27 1.27)) hide)
     )
-    (pin "1")
-    (pin "2")
-  )
-  (symbol (lib_id "localstuff:C") (at 124.46 36.83 0) (unit 1)
+    (property "LCSC" "C70225" (id 4) (at 146.05 36.83 0)
+      (effects (font (size 1.27 1.27)))
+    )
+    (pin "1")
+    (pin "2")
+  )
+  (symbol (lib_id "localparts:CP_100n_50V_0603") (at 124.46 36.83 0) (unit 1)
     (in_bom yes) (on_board yes)
     (property "Reference" "C1" (id 0) (at 125.095 34.29 0)
@@
       (effects (font (size 1.27 1.27)) (justify left))
     )
-    (property "Footprint" "Capacitor_SMD:C_0603_1608Metric_Pad1.05x0.95mm_HandSolder" (id 2) (at 125.4252 40.64 0)
+    (property "Footprint" "Capacitor_SMD:C_0603_1608Metric" (id 2) (at 125.4252 40.64 0)
       (effects (font (size 1.27 1.27)) hide)
     )
     (property "Datasheet" "" (id 3) (at 124.46 36.83 0)
       (effects (font (size 1.27 1.27)) hide)
+    )
+    (property "LCSC" "C14663" (id 4) (at 124.46 36.83 0)
+      (effects (font (size 1.27 1.27)))
     )
     (pin "1")
@@
     (pin "2")
   )
-  (symbol (lib_id "localstuff:CP") (at 236.22 45.72 0) (unit 1)
-    (in_bom yes) (on_board yes)
+  (symbol (lib_id "localparts:CP_100n_50V_0603") (at 236.22 45.72 0) (unit 1)
+    (in_bom no) (on_board no)
     (property "Reference" "C6" (id 0) (at 229.87 43.18 0)
       (effects (font (size 1.27 1.27)) (justify left))
@@
     (property "Datasheet" "" (id 3) (at 236.22 45.72 0)
       (effects (font (size 1.27 1.27)) hide)
+    )
+    (property "LCSC" "C14663" (id 4) (at 236.22 45.72 0)
+      (effects (font (size 1.27 1.27)))
     )
     (pin "1")
@@
   )
   (symbol (lib_name "LTC4311_1") (lib_id "localstuff:LTC4311") (at 186.69 45.72 0) (unit 1)
-    (in_bom yes) (on_board yes) (fields_autoplaced)
+    (in_bom no) (on_board no) (fields_autoplaced)
     (property "Reference" "U3" (id 0) (at 199.39 38.2144 0)
       (effects (font (size 1.524 1.524)))
@@
   )
   (symbol (lib_id "localstuff:LTC4311") (at 212.09 45.72 0) (mirror y) (unit 1)
-    (in_bom yes) (on_board yes) (fields_autoplaced)
+    (in_bom no) (on_board no) (fields_autoplaced)
     (property "Reference" "U4" (id 0) (at 212.6106 34.29 0)
       (effects (font (size 1.524 1.524)) (justify right))
@@
     (pin "9")
   )
-  (symbol (lib_id "localstuff:CP") (at 45.72 109.22 0) (unit 1)
+  (symbol (lib_id "localparts:CP_1µ_50V_0603") (at 45.72 109.22 0) (unit 1)
     (in_bom yes) (on_board yes)
     (property "Reference" "C4" (id 0) (at 39.37 106.68 0)
@@
       (effects (font (size 1.27 1.27)) (justify left))
     )
-    (property "Footprint" "Capacitor_SMD:C_0603_1608Metric" (id 2) (at 46.6852 113.03 0)
-      (effects (font (size 1.27 1.27)) hide)
-    )
-    (property "Datasheet" "" (id 3) (at 45.72 109.22 0)
-      (effects (font (size 1.27 1.27)) hide)
+    (property "Footprint" "Resistor_SMD:R_0603_1608Metric_Pad0.98x0.95mm_HandSolder" (id 2) (at 49.53 108.2548 0)
+      (effects (font (size 1.27 1.27)) hide)
+    )
+    (property "Datasheet" "~" (id 3) (at 45.72 109.22 0)
+      (effects (font (size 1.27 1.27)) hide)
+    )
+    (property "LCSC" "C15849" (id 4) (at 45.72 109.22 0)
+      (effects (font (size 1.27 1.27)))
     )
     (pin "1")
@@
     (pin "1")
   )
-  (symbol (lib_id "localstuff:CP") (at 77.47 109.22 0) (unit 1)
+  (symbol (lib_id "localparts:CP_1µ_50V_0603") (at 77.47 109.22 0) (unit 1)
     (in_bom yes) (on_board yes) (fields_autoplaced)
     (property "Reference" "C5" (id 0) (at 81.28 107.0609 0)
@@
       (effects (font (size 1.27 1.27)) (justify left))
     )
-    (property "Footprint" "Capacitor_SMD:C_0603_1608Metric" (id 2) (at 78.4352 113.03 0)
-      (effects (font (size 1.27 1.27)) hide)
-    )
-    (property "Datasheet" "" (id 3) (at 77.47 109.22 0)
-      (effects (font (size 1.27 1.27)) hide)
+    (property "Footprint" "Resistor_SMD:R_0603_1608Metric_Pad0.98x0.95mm_HandSolder" (id 2) (at 81.28 108.2548 0)
+      (effects (font (size 1.27 1.27)) hide)
+    )
+    (property "Datasheet" "~" (id 3) (at 77.47 109.22 0)
+      (effects (font (size 1.27 1.27)) hide)
+    )
+    (property "LCSC" "C15849" (id 4) (at 77.47 109.22 0)
+      (effects (font (size 1.27 1.27)))
     )
     (pin "1")
@@
     )
     (path "/00000000-0000-0000-0000-00005dd291db"
-      (reference "C1") (unit 1) (value "100nF") (footprint "Capacitor_SMD:C_0603_1608Metric_Pad1.05x0.95mm_HandSolder")
+      (reference "C1") (unit 1) (value "100nF") (footprint "Capacitor_SMD:C_0603_1608Metric")
     )
     (path "/00000000-0000-0000-0000-00005baeabab"
-      (reference "C2") (unit 1) (value "100nF") (footprint "Capacitor_SMD:C_0603_1608Metric_Pad1.05x0.95mm_HandSolder")
+      (reference "C2") (unit 1) (value "100nF") (footprint "Capacitor_SMD:C_0603_1608Metric")
     )
     (path "/00000000-0000-0000-0000-00005dcd465c"
-      (reference "C3") (unit 1) (value "10µF") (footprint "Capacitor_SMD:C_1206_3216Metric_Pad1.42x1.75mm_HandSolder")
+      (reference "C3") (unit 1) (value "10µF") (footprint "Capacitor_SMD:C_0603_1608Metric")
     )
     (path "/9bb18cf9-3331-4cf8-baa7-8b523620c000"
-      (reference "C4") (unit 1) (value "1µF") (footprint "Capacitor_SMD:C_0603_1608Metric")
+      (reference "C4") (unit 1) (value "1µF") (footprint "Resistor_SMD:R_0603_1608Metric_Pad0.98x0.95mm_HandSolder")
     )
     (path "/d274b249-30d2-4700-a710-2d78efb57ae4"
-      (reference "C5") (unit 1) (value "1µF") (footprint "Capacitor_SMD:C_0603_1608Metric")
+      (reference "C5") (unit 1) (value "1µF") (footprint "Resistor_SMD:R_0603_1608Metric_Pad0.98x0.95mm_HandSolder")
     )
     (path "/4820f679-3ab4-4bd9-8d32-15992367d578"
