File: misc/solvis-control/solvis-control.kicad_pcb (KiCad board)
At the start: 2 copper layers, 54.4 x 45.9 mm, 22 parts, among them J1 Conn_01x04_Socket, Q1 SI2390DS, Q2 2N7002, U1 MOC8101, U3 CPC1965G, U4 CPC1965G, U5 CPC1965G

Commit message: Old check-in: solvis-control
Parts:
- removed JPUMP1: Conn_01x03_Socket, localstuff:Würth3.5mm_3
- removed JSWITCH1: Conn_01x04_Socket, localstuff:Würth3.5mm_4
- added C3: CP_1µ_0603, Capacitor_SMD:C_0603_1608Metric, F.Cu at (85.6, 60.7)
- added C4: CP_100n_50V_0603, Capacitor_SMD:C_0603_1608Metric, F.Cu at (80.4, 38.7)
- added C5: CP_100n_50V_0603, Capacitor_SMD:C_0603_1608Metric, F.Cu at (80.4, 54.4)
- added C6: CP_100n_50V_0603, Capacitor_SMD:C_0603_1608Metric, F.Cu at (80.4, 62.0)
- added C7: CP_100n_50V_0603, Capacitor_SMD:C_0603_1608Metric, F.Cu at (80.4, 46.2)
- added C8: C_1µ_25V_0603, Capacitor_SMD:C_0603_1608Metric, F.Cu at (91.5, 47.5)
- added J2: Conn_01x04_Socket, Connector_JST:JST_PH_B4B-PH-K_1x04_P2.00mm_Vertical, F.Cu at (73.9, 66.7)
- added JSW_BUFFER_SWITCH1: Conn_01x03_Socket, localstuff:Würth3.5mm_3, F.Cu at (122.7, 58.0)
- added JSW_HEAT_VALVE1: Conn_01x04_Socket, localstuff:Würth3.5mm_4, F.Cu at (122.6, 38.2)
- added JSW_SOLVIS_VALVE1: Conn_01x03_Socket, localstuff:Würth3.5mm_3, F.Cu at (122.7, 72.2)
- added J_12V2: Conn_01x02, localstuff:1X02_GN, F.Cu at (74.8, 73.5)
- added J_TP1: Conn_01x02, localstuff:1X02_GN, F.Cu at (74.7, 60.1)
- added J_TP2: Conn_01x02, localstuff:1X02_GN, F.Cu at (74.7, 52.2)
- added J_TP3: Conn_01x02, localstuff:1X02_GN, F.Cu at (74.7, 44.4)
- added J_TP4: Conn_01x02, localstuff:1X02_GN, F.Cu at (74.7, 36.6)
- added Q3: 2N7002, Package_TO_SOT_SMD:SOT-23, F.Cu at (93.6, 50.1)
- added R10: R_360_0603, Resistor_SMD:R_0603_1608Metric_Pad0.98x0.95mm_HandSolder, F.Cu at (91.9, 54.4)
- added R11: R_1k_0603, Resistor_SMD:R_0603_1608Metric, F.Cu at (88.4, 61.4)
- added R12: R_1k_0603, Resistor_SMD:R_0603_1608Metric, F.Cu at (85.6, 62.5)
- added R13: R_1k_0603, Resistor_SMD:R_0603_1608Metric, F.Cu at (85.6, 64.2)
- added R14: R_1k_0603, Resistor_SMD:R_0603_1608Metric, F.Cu at (80.4, 59.0)
- added R15: R_1k_0603, Resistor_SMD:R_0603_1608Metric, F.Cu at (80.4, 51.4)
- added R16: R_1k_0603, Resistor_SMD:R_0603_1608Metric, F.Cu at (80.4, 43.2)
- added R17: R_1k_0603, Resistor_SMD:R_0603_1608Metric, F.Cu at (80.4, 35.7)
- added R18: R_1k_0603, Resistor_SMD:R_0603_1608Metric, F.Cu at (82.8, 61.4)
- added R8: R 100k, Resistor_SMD:R_0603_1608Metric_Pad0.98x0.95mm_HandSolder, F.Cu at (90.8, 50.2)
- added R9: R_360_0603, Resistor_SMD:R_0603_1608Metric_Pad0.98x0.95mm_HandSolder, F.Cu at (91.8, 52.8)
- added U6: CPC1965G, localstuff:DIL16-CPC1965G, F.Cu at (106.9, 38.9)
- added U7: CPC1965G, localstuff:DIL16-CPC1965G, F.Cu at (106.9, 49.0)
- added U8: MCP3428x-xSL, Package_SO:SOIC-14_3.9x8.7mm_P1.27mm, F.Cu at (85.4, 55.1)
- added U9: AZ1117-3.3, Package_TO_SOT_SMD:SOT-223, F.Cu at (85.9, 46.0)
- J1: footprint Connector_JST:JST_PH_B4B-PH-K_1x04_P2.00mm_Vertical -> localstuff:RJ11
- R4, R5, R6: value R_100_0603 -> R_360_0603
- moved R2 27.8 mm to (90.7, 44.0)
- moved Q1 27.7 mm to (93.5, 43.9)
- moved J_12V1 25.4 mm to (92.6, 36.9), turned to 0 degrees
- moved J_PWM1 20.9 mm to (85.2, 36.9), turned to 0 degrees
- moved C2 13.6 mm to (100.1, 83.3), turned to 90 degrees
- moved J1 6.94 mm to (104.2, 94.2), turned to 180 degrees
- moved R3 4.60 mm to (81.1, 75.6)
- moved R7 3.82 mm to (91.0, 57.0), turned to -90 degrees
- moved U3 1.10 mm to (107.0, 59.1)
- moved U4 0.60 mm to (106.9, 69.2)
Connections:
- C2 pad 1: /V33 -> +3.3V
- J1 pad 4: /V33 -> +3.3V
- J_230V1 pad 1: Net-(JPUMP1-Pin_3) -> /L
- J_230V1 pad 2: Net-(JPUMP1-Pin_2) -> /N
- J_230V1 pad 3: Net-(J_230V1-Pin_3) -> /PE
- U2 pad 10: unconnected-(U2-GPIO9-Pad10) -> /SCL
- U2 pad 21: unconnected-(U2-3V3-Pad21) -> +3.3V
- U2 pad 23: /V33 -> unconnected-(U2-VBUS-Pad23)
- U2 pad 7: unconnected-(U2-GPIO6-Pad7) -> Net-(U2-GPIO6)
- U2 pad 8: unconnected-(U2-GPIO7-Pad8) -> Net-(Q3-G)
- U2 pad 9: unconnected-(U2-GPIO8-Pad9) -> /SDA
- U3 pad 10: Net-(J_230V1-Pin_3) -> /L
- U4 pad 10: Net-(J_230V1-Pin_3) -> /L
- U5 pad 10: Net-(J_230V1-Pin_3) -> /L
Routing:
- net /PE: track 0.00 -> 311.5 mm
- net Net-(JPUMP1-Pin_2): track 241.4 -> 0.00 mm
- net +3.3V: track 0.00 -> 151.9 mm, vias 0 -> 7
- net GND: track 70.1 -> 175.2 mm, vias 12 -> 32
- net Net-(J_230V1-Pin_3): track 89.1 -> 0.00 mm
- net /V33: track 66.6 -> 0.00 mm
- net /N: track 0.00 -> 60.5 mm
- net /L: track 0.00 -> 59.6 mm
- net Net-(U2-GPIO6): track 0.00 -> 45.7 mm, vias 0 -> 4
- net Net-(Q3-G): track 0.00 -> 44.2 mm, vias 0 -> 2
- net /SCL: track 0.00 -> 42.4 mm, vias 0 -> 3
- net +12V: track 0.00 -> 40.3 mm, vias 0 -> 3
- net /SDA: track 0.00 -> 37.1 mm, vias 0 -> 2
- net Net-(J_TP4-Pin_2): track 0.00 -> 28.3 mm, vias 0 -> 2
- net /ADCREF: track 0.00 -> 24.7 mm, vias 0 -> 5
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Other:
- board size 54.4 x 45.9 mm -> 54.4 x 67 mm
- board text added: "CP_100n_50V_0603"
- board text added: "R18"
