File: misc/solvis-control/solvis-control.kicad_sch (KiCad schematic)
At the start: 22 parts, among them J1 Conn_01x04_Socket, Q1 SI2390DS, Q2 2N7002, U1 MOC8101, U3 CPC1965G, U4 CPC1965G, U5 CPC1965G

Commit message: Old check-in: solvis-control
Parts:
- added C3: CP_1µ_0603, Capacitor_SMD:C_0603_1608Metric, symbol localparts:CP_1µ_25V_0603
- added C4, C5, C6, C7: CP_100n_50V_0603, Capacitor_SMD:C_0603_1608Metric, symbol localparts:CP_100n_50V_0603
- added C8: C_1µ_25V_0603, Capacitor_SMD:C_0603_1608Metric, symbol localparts:CP_1µ_25V_0603
- added J2: Conn_01x04_Socket, Connector_JST:JST_PH_B4B-PH-K_1x04_P2.00mm_Vertical, symbol Connector:Conn_01x04_Socket
- added JSW_HEAT_VALVE1: Conn_01x04_Socket, localstuff:Würth3.5mm_4, symbol Connector:Conn_01x04_Socket
- added J_12V2, J_TP1, J_TP2, J_TP3, J_TP4: Conn_01x02, localstuff:1X02_GN, symbol Connector_Generic:Conn_01x02
- added Q3: 2N7002, Package_TO_SOT_SMD:SOT-23, symbol localstuff:2N7002
- added R10, R9: R_360_0603, Resistor_SMD:R_0603_1608Metric_Pad0.98x0.95mm_HandSolder, symbol localparts:R_100_0603
- added R11, R12, R13, R14, R15, R16, R17, R18: R_1k_0603, Resistor_SMD:R_0603_1608Metric, symbol localparts:R_1k_0603
- added R8: R 100k, Resistor_SMD:R_0603_1608Metric_Pad0.98x0.95mm_HandSolder, symbol Device:R
- added U6, U7: CPC1965G, localstuff:DIL16-CPC1965G, symbol localstuff:CPC1965G
- added U8: MCP3428x-xSL, Package_SO:SOIC-14_3.9x8.7mm_P1.27mm, symbol Analog_ADC:MCP3428x-xSL
- added U9: AZ1117-3.3, Package_TO_SOT_SMD:SOT-223, symbol localstuff:AZ1117-3V3
- J1: footprint Connector_JST:JST_PH_B4B-PH-K_1x04_P2.00mm_Vertical -> localstuff:RJ11
- JSW_BUFFER_SWITCH1: renamed from JSWITCH1; value Conn_01x04_Socket -> Conn_01x03_Socket; footprint localstuff:Würth3.5mm_4 -> localstuff:Würth3.5mm_3; symbol Connector:Conn_01x04_Socket -> Connector:Conn_01x03_Socket
- R4, R5: value R_100_0603 -> R_360_0603; Bin b-r-100-s -> b-r-360-s; Display 100 Ω -> 360 Ω; LCSC C22775 -> (none)
- R6: value R_100_0603 -> R_360_0603; Bin b-r-100-s -> b-r-360-s; Display 100 Ω -> 360 Ω
- renumbered JPUMP1 to JSW_SOLVIS_VALVE1
Connections:
- net GND: now also C3.2, C4.2, C5.2, C6.2, C7.2, C8.2, J2.1 (Pin_1), J_12V2.1 (Pin_1), J_TP1.1 (Pin_1), J_TP2.1 (Pin_1), J_TP3.1 (Pin_1), J_TP4.1 (Pin_1), Q3.2 (S), R13.2, R8.2, U6.1 (-), U7.1 (-), U8.10 (Adr1), U8.5 (V_{SS}), U8.9 (Adr0), U9.1 (ADJ)
- net L: now reaches U3.10 (A1), U4.10 (A1), U5.10 (A1)
- net L: now also J_230V1.1 (Pin_1), U6.10 (A1), U7.10 (A1); no longer J_230V1.3 (Pin_3)
- net SCL: now reaches U2.10 (GPIO9)
- net SCL: now also J2.3 (Pin_3), R11.1, U8.8 (SCL)
- net +3.3V: now reaches U2.21 (3V3)
- net +3.3V: now also C2.1, J1.4 (Pin_4), C3.1, J2.4 (Pin_4), R11.2, R12.1, R14.2, R15.1, R16.2, R17.1, R18.2, U8.6 (V_{DD})
- net at U2.7 (GPIO6): now also R9.2
- net at U2.8 (GPIO7): now also Q3.1 (G), R10.2, R8.1
- net SDA: now reaches U2.9 (GPIO8)
- net SDA: now also J2.2 (Pin_2), R18.1, U8.7 (SDA)
- net N: now reaches JSW_BUFFER_SWITCH1.3 (Pin_3), JSW_SOLVIS_VALVE1.2 (Pin_2), J_230V1.2 (Pin_2)
- net N: now also JSW_HEAT_VALVE1.3 (Pin_3)
- removed net V33: C2.1, J1.4 (Pin_4), U2.23 (VBUS)
- new net: C4.1, J_TP4.2 (Pin_2), R17.2, U8.13 (CH4+)
- new net: JSW_HEAT_VALVE1.1 (Pin_1), U6.8 (A2)
- new net: JSW_HEAT_VALVE1.2 (Pin_2), U7.8 (A2)
- new net: R10.1, U7.16 (+)
- new net: C7.1, J_TP3.2 (Pin_2), R16.1, U8.11 (CH3+)
- new net: Q3.3 (D), R9.1, U6.16 (+)
- new net: C6.1, J_TP1.2 (Pin_2), R14.1, U8.1 (CH1+)
- new net: C5.1, J_TP2.2 (Pin_2), R15.2, U8.3 (CH2+)
- new net +12V: J_12V2.2 (Pin_2), U9.3 (VI)
- new net +3V3: C8.1, U9.2 (VO)
- new net ADCREF: R12.2, R13.1, U8.12 (CH3-), U8.14 (CH4-), U8.2 (CH1-), U8.4 (CH2-)
- new net PE: JSW_HEAT_VALVE1.4 (Pin_4), JSW_SOLVIS_VALVE1.3 (Pin_3), J_230V1.3 (Pin_3)
Other:
- moved on the sheet: C1, C2, J1, JSW_SOLVIS_VALVE1, J_230V1, J_IN1, J_OUT1, Q1, Q2, R1, R2, R3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
