File: bms/base18/base18.kicad_sch (KiCad schematic)
At the start: 171 parts, among them J1 Conn_LEM_3, J10 Conn_02x11_Odd_Even, J11 Conn_01x10, J12 Conn_01x09, J13 Conn_01x04, J14 Conn_01x03_Socket, J2 Conn_LEM_5, J3 Conn_01x02_Female, J4 Conn_01x04, J5 Conn_01x04, J6 Conn_01x02_Female, J7 Conn_01x20, J8 Conn_02x12_Odd_Even, J9 Conn_02x04_Odd_Even, Q1 DMN2058U-7, Q10 DMP2035U, Q11 DMP2035U, Q12 DMP2035U, Q13 DMP2035U, Q14 DMP2035U, Q15 DMP2035U, Q16 DMP2035U, Q17 DMP2035U, Q18 DMP2035U, Q19 DMP2035U, Q2 DMN2058U, Q20 DMP2035U, Q21 DMP2035U, Q3 DMP2035U, Q4 DMP2035U, Q5 DMP2035U, Q6 DMP2035U, Q7 DMP2035U, Q8 DMP2035U, Q9 DMP2035U, U1 TSR_1-48120WI, U10 ESP32-WROOM, U11 LT1785xS8, U12 AZ1117-3.3, U2 STH05_12, U3 ADBMS1818, U4 Pico, U5 AZ1117-5.0, U6 MCP2562-E-SN, U7 MCP2515-xSO, U8 4051, U9 4051

Commit message: some update
Parts:
- C1: LCSC C5250958 -> C72488
- C2: JLCPosOffset (none) -> -6.15,0; JLCRotOffset (none) -> 180
- C27: Display 10µF 100V -> 1µF 100V; LCSC C2171077 -> C385977
- C40, C42, C44: Display 100 nF -> 100 nF 50V
- D1: footprint localstuff:SOD-123FL -> Diode_SMD:D_SMB
- D2: footprint Diode_SMD:D_SOD-523 -> Diode_SMD:D_SOD-123
- J1: JLCPosOffset (none) -> -4,0; JLCRotOffset (none) -> 180; LCSC (none) -> C157993
- J10: JLCPosOffset (none) -> 10,1; JLCRotOffset (none) -> -90
- J11: JLCPosOffset (none) -> 9,0; JLCRotOffset (none) -> -90; LCSC C468242 -> C158038
- J12: JLCPosOffset (none) -> -8,0; JLCRotOffset (none) -> 90; LCSC C545753 -> C157968
- J2: JLCPosOffset (none) -> -3,0; JLCRotOffset (none) -> 180; LCSC (none) -> C131334
- Q1: value DMN2058U-7 -> DMN2058U; symbol localparts:Q_NMOS_20V_4A_lowVth -> localstuff:DMN2058U; JLCRotOffset (none) -> 180; LCSC C2760648 -> C461001
- Q10, Q11, Q12, Q13, Q14, Q15, Q16, Q17, Q18, Q19, Q20, Q3, Q4, Q5, Q6, Q7, Q8, Q9: symbol localparts:DMP2035U -> localstuff:DMP2035U; JLCRotOffset (none) -> 180; LCSC (none) -> C110499
- Q2: JLCRotOffset (none) -> 180; LCSC C2760648 -> C461001
- Q21, U12: JLCRotOffset (none) -> 180
- R13, R16, R19, R22, R25, R28, R31, R34, R37, R40, R43, R46, R49, R52, R55, R58, R7, R9: footprint localstuff:R_Radial_Power_D11.0mm -> localstuff:R_Radial_Power_L12.5mm_W9.0mm_P5.00mm; JLCRotOffset (none) -> 90
- U10: JLCPosOffset (none) -> 1,0; JLCRotOffset (none) -> -90
- U11, U5, U7, U8, U9: JLCRotOffset (none) -> -90
- U3: footprint Package_DFN_QFN:QFN-64-1EP_9x9mm_P0.5mm_EP5.45x5.45mm_ThermalVias -> Package_QFP:LQFP-64-1EP_10x10mm_P0.5mm_EP5x5mm_ThermalVias; JLCRotOffset (none) -> 90; LCSC C3682393 -> C2971928
- U6: symbol Interface_CAN_LIN:MCP2562-E-SN -> localparts:MCP2562-E-SN; JLCRotOffset (none) -> -90; LCSC (none) -> C53609

Commit message: Old check-in: base18
Parts:
- J11: Farnell (none) -> 1830772
- J12: Farnell (none) -> 1830771
Changed lines of the file:
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@@
       (effects (font (size 1.27 1.27)) hide)
     )
+    (property "Farnell" "1830771" (at 27.94 34.29 90)
+      (effects (font (size 1.27 1.27)) hide)
+    )
     (pin "1")
     (pin "2")
@@
       (effects (font (size 1.27 1.27)) hide)
     )
+    (property "Farnell" "1830772" (at 27.94 57.15 90)
+      (effects (font (size 1.27 1.27)) hide)
+    )
