File: misc/usb-int/usb-int-pi.kicad_pcb (KiCad board)
At the start: 2 copper layers, 22.7 x 17.4 mm, 16 parts, among them J1 USB_A_Device, J2 USB_A_Host, J3 Conn_01x04_Pin, U2 AP2151W, U3 FSUSB42MUX, U4 TPS78233DDC

Commit message: Old check-in: usb-int
Parts:
- J2: footprint Connector_USB:USB_A_Stewart_SS-52100-001_Horizontal -> localstuff:USB_A_Stewart_SS-52100-001_Horizontal
Changed lines of the file:
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@@
       (net 7 "GNDPWR") (pinfunction "Shield") (pintype "passive"))
     (model "${moat3d}/USB-AM-S-X-X-TH.step"
-      (offset (xyz 0 -8.4 0))
+      (offset (xyz 0 -8.4 -1.5))
       (scale (xyz 1 1 1))
       (rotate (xyz -90 0 0))
     )
   )
-  (footprint "Connector_USB:USB_A_Stewart_SS-52100-001_Horizontal" (layer "B.Cu")
+  (footprint "localstuff:USB_A_Stewart_SS-52100-001_Horizontal" (layer "B.Cu")
     (at 132.81 112.875 -90)
     (descr "USB A connector https://belfuse.com/resources/drawings/stewartconnector/dr-stw-ss-52100-001.pdf")
@@
     (property "ki_keywords" "connector USB")
     (attr through_hole)
-    (fp_text reference "J2" (at 11.125 0.21 unlocked) (layer "F.SilkS")
-        (effects (font (size 0.8 0.8) (thickness 0.12)))
+    (fp_text reference "J2" (at 3.5 2.26 90) (layer "B.SilkS")
+        (effects (font (size 1 1) (thickness 0.15)) (justify mirror))
     )
     (fp_text value "USB_A_Host" (at 3.5 -14.49 90) (layer "B.Fab")
@@
     (pad "5" thru_hole circle (at 10.07 -2.71 270) (size 3 3) (drill 2.3) (layers "*.Cu" "*.Mask")
       (net 7 "GNDPWR") (pinfunction "Shield") (pintype "passive"))
-    (model "${KICAD6_3DMODEL_DIR}/Connector_USB.3dshapes/USB_A_Stewart_SS-52100-001_Horizontal.wrl"
-      (offset (xyz 0 0 0))
+    (model "${moat3d}/SS-52100-001.stp"
+      (offset (xyz 3.5 -6 4))
       (scale (xyz 1 1 1))
-      (rotate (xyz 0 0 0))
+      (rotate (xyz 180 0 180))
     )
   )
