File: misc/thermo/thermo.kicad_pcb (KiCad board)
At the start: 2 copper layers, 44.5 x 60.6 mm, 21 parts, among them J1 Conn_01x04_Pin, J2 Conn_01x04_Pin, J3 Conn_01x04_Pin, Q1 2N7002, U1 CPC1965G, U2 ESP-12S

Commit message: Update thermo
Parts:
- added G***: LOGO, localstuff:OSHW Logo 3mm Cu, B.Cu at (123.4, 73.3)
- added J4: Conn_01x04_Pin, Connector_PinHeader_2.54mm:PinHeader_1x04_P2.54mm_Vertical, F.Cu at (155.4, 72.3)
- G***: moved to F.Cu
- J1, J2, J3: footprint Connector_JST:JST_XH_B4B-XH-A_1x04_P2.50mm_Vertical -> Connector_JST:JST_SH_BM04B-SRSS-TB_1x04-1MP_P1.00mm_Vertical
- moved J3 6.13 mm to (144.6, 68.2), turned to 90 degrees
- moved J1 5.50 mm to (150.5, 68.2)
- moved J2 3.66 mm to (138.7, 68.2), turned to 90 degrees
- moved G*** 1.30 mm to (123.4, 73.3), turned to 0 degrees
Connections:
- J2 pad 3: SCL -> SDA
- J2 pad 4: SDA -> SCL
- J3 pad 3: SCL -> SDA
- J3 pad 4: SDA -> SCL
Routing:
- net SDA: track 32.8 -> 38.9 mm, vias 0 -> 2
- net +3V3: track 110.4 -> 107.9 mm, vias 1 -> 2
- net GND: track 109.3 -> 111.6 mm, vias 13 -> 16
- net Net-(J_PWR1-Pin_2): track 59.8 -> 57.7 mm
- net Net-(U1-+): track 30.0 -> 30.9 mm
- net SCL: track 42.2 -> 43.0 mm, vias 1 -> 2
Other:
- board text added: "Thermo Switch MoaT V1.2"
- board text removed: "Thermo Switch"
- board text removed: "V1.1 MoaT"
