File: misc/gaggenau/gaggenau.kicad_sch (KiCad schematic)
At the start: 97 parts, among them IC1 ESP32-C6-WROOM-1-N8, J1 Mains, J10 VentX, J2 Vent, J3 Conn_01x08_Socket, J4 Light, J5 MCU, J6 MCU, J7 ?, J8 ? Klemmen, J9 Conn_02x04_Odd_Even, K1 Relay_SPDT, Q1 BC547, Q10 Q_PMOS, Q11 Q_PMOS, Q12 Q_PMOS, Q13 Q_PMOS, Q14 Q_NMOS, Q2 BTB16-600BW, Q3 BC547, Q4 BC547, Q5 BC547, Q6 BC547, Q7 BC547, Q8 BC547, Q9 Q_NMOS, SW1 L1, SW2 L0, SW3 L2, SW4 L3, SW5 Int, SW6 Timer, SW7 Licht, SW8 F, U1 PC-817, U2 MC33064P, U3 93C06C, U4 KMOC302S, U5 CPC1965G, Y1 Crystal_GND2

Commit message: Save: Gaggenau v1
Connections:
- net L: now also C1.2, J1.3 (Pin_3), L1.1, PS1.1 (L)
- net N: now also C1.1, J1.2 (Pin_2), L1.3, PS1.2 (N)
Changed lines of the file:
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@@
 		)
 	)
+	(label "L"
+		(at 25.4 26.67 0)
+		(effects
+			(font
+				(size 1.27 1.27)
+			)
+			(justify left bottom)
+		)
+	)
 	(label "PA5"
 		(at 133.35 127 0)
@@
 		)
 	)
+	(label "N"
+		(at 25.4 24.13 0)
+		(effects
+			(font
+				(size 1.27 1.27)
+			)
+			(justify left bottom)
+		)
+	)
 	(label "PA4"
 		(at 133.35 124.46 0)
@@
 		)
 		(property "Display" "10 kΩ"
-			(at 147.32 114.3 0)
+			(at 147.828 118.872 90)
 			(effects
 				(font

Commit message: Gaggenau replacement v2
Parts:
- removed U1: PC-817, Package_DIP:SMDIP-4_W9.53mm, symbol Isolator:PC817
- added C19: 22nF 400V X2, Capacitor_THT:C_Rect_L11.0mm_W5.1mm_P10.00mm_MKT, symbol Device:C
- added C20: 100nF, Capacitor_SMD:C_0402_1005Metric, symbol localparts:CP_10µ_16V_0603
- added C21: 22µF, Capacitor_SMD:C_1206_3216Metric, symbol localparts:CP_10µ_16V_0603
- added D6: ESDA041, Diode_SMD:D_SOD-323, symbol Diode:1.5KExxA
- added F1, F2: FuseHolder, Fuse:Fuseholder_Cylinder-5x20mm_Stelvio-Kontek_PTF78_Horizontal_Open, symbol localstuff:FuseHolder
- added R31, R33: 470 100V, Resistor_SMD:R_2512_6332Metric, symbol Device:R
- added R32: 2k2, Resistor_SMD:R_2512_6332Metric, symbol Device:R
- added R34: 22k, Resistor_THT:R_Axial_DIN0309_L9.0mm_D3.2mm_P15.24mm_Horizontal, symbol Device:R
- added R35: 47k, Resistor_SMD:R_0603_1608Metric, symbol localparts:R_47k_0603
- added R36, R37: 1M, Resistor_THT:R_Axial_DIN0204_L3.6mm_D1.6mm_P5.08mm_Horizontal, symbol localparts:R_100k_0603
- added RV1: Varistor230V, localstuff:Varistor_Disc_D21mm_W10mm_P7.5mm, symbol localparts:Varistor230V
- added U1: PC814, Package_DIP:SMDIP-4_W9.53mm, symbol localparts:PC814
- added U6: PC-817, Package_DIP:SMDIP-4_W9.53mm, symbol Isolator:PC817
- C16: value 10µF -> 10nF; Bin b-c-10u-s8 -> (none); Display 10 µF 16V -> 10nF; LCSC C1691 -> C1589
- D2: now left out of the parts list
- PS1: value RAC01-3.3 -> Apos03; footprint localstuff:RAC01-3.3 -> localstuff:Hiecube AP05-Zero; symbol localstuff:RAC01-3.3 -> localstuff:Apos03; LCSC (none) -> C432582; MANUFACTURER Vigortronix -> Hiecube; now in the parts list
- Prog1: LCSC (none) -> C2685197; now in the parts list
- R1: value 22k -> 2k2; footprint Resistor_THT:R_Axial_DIN0309_L9.0mm_D3.2mm_P15.24mm_Horizontal -> Resistor_SMD:R_2512_6332Metric; LCSC C61349 -> C421608
Connections:
- net Btn5: now also IC1.4 (IO4); no longer IC1.11 (IO10)
- net Btn6: now also IC1.5 (IO5); no longer IC1.12 (IO11)
- net Btn7: now also IC1.6 (IO6); no longer IC1.13 (IO12)
- net Btn8: now also IC1.7 (IO7); no longer IC1.14 (IO13)
- net EN: now also C16.1
- net Earth_Protective: now also R36.2; no longer C10.2, C11.2, C12.2, C17.2, C18.2
- net GND: now also C10.2, C11.2, C12.2, C16.2, C17.2, C18.2, PS1.4 (DC-), C20.2, C21.2, D6.2 (A2), R37.1, U1.3, U6.3; no longer C16.1, PS1.3 (DC-)
- net Ivent: now also R35.2, U1.4, U6.4
- net L: now also F1.2, F2.2, R34.1; no longer C1.2, C3.2, C4.2, L1.1, L1.2, PS1.1 (L), Q2.1 (A1), R1.1, TR1.4, U5.8 (A2)
- net Llight: now also J4.2 (Pin_2); no longer J4.1 (Pin_1)
- net N: now also J4.1 (Pin_1), L1.1, R1.1, RV1.2, U6.2; no longer C2.1, C4.1, J10.2 (Pin_2), J2.2 (Pin_2), J4.2 (Pin_2), L1.3, L1.4, TR1.5
- net VCC: now also PS1.3 (DC+), R22.1, C20.1, C21.1, D6.1 (A1), R35.1; no longer C16.2, PS1.4 (DC+), R22.2
- net at IC1.10 (IO8): now also R22.2; no longer R22.1
- net at R1.2: now also R32.1; no longer D2.2 (A)
- net at D2.1 (K): now also U6.1
- new net: R31.2, R33.1
- new net: C1.2, F2.1, L1.3
- new net: R32.2, U1.1
- new net: R36.1, R37.2
- new net: D2.2 (A), R34.2
- new net: C19.2, R33.2, U1.2
- new net Lf: C19.1, F1.1, PS1.1 (L), R31.1, RV1.1, U5.8 (A2)
- new net Lx: C3.2, C4.2, L1.4, Q2.1 (A1), TR1.4
- new net Nx: C2.1, C4.1, J10.2 (Pin_2), J2.2 (Pin_2), L1.2, TR1.5
- no-connect marks 3 -> 2
Other:
- note added: "Phase Sensor, old"
- moved on the sheet: D2, R21, R22, R5

Commit message: Gaggenau controller update
Parts:
- removed C15: C_Small, symbol Device:C_Small
- added D7: SMAJ5.0CA, Diode_SMD:D_SMA, symbol Diode:SMAJ5.0CA
- added R38: 220, Resistor_SMD:R_0603_1608Metric, symbol Device:R
- C19: value 22nF 400V X2 -> 220nF 400V X2; LCSC C390050 -> C489075
- D6: value ESDA041 -> P6KE6.8A
- J10: value VentX -> Cap
- R1, R32: value 2k2 -> 27; footprint Resistor_SMD:R_2512_6332Metric -> Resistor_SMD:R_1206_3216Metric; LCSC C421608 -> C25367
- R31: value 470 100V -> 470k 200V
- R33: value 470 100V -> 470k 100V
Connections:
- net Btn6: no longer C11.1, J3.7 (Pin_7), J9.5 (Pin_5), R17.2, R30.1, SW3.3 (K), SW5.3 (K), SW7.3 (K)
- net Lf: no longer C19.1, R31.1
- net Lf2: now reaches C1.2, F2.1, L1.3
- net Lf2: now also C19.1, R31.1
- net at R32.2: now also D7.2 (A2), R38.2; no longer U1.1
- net at C19.2, R33.2, U1.2: now also D7.1 (A1)
- new net: R38.1, U1.1
- new net Kbraun: C11.1, J3.7 (Pin_7), J9.5 (Pin_5), R17.2, R30.1, SW3.3 (K), SW5.3 (K), SW7.3 (K)
Other:
- moved on the sheet: C1, Q3, Q4, Q5, Q6, Q7, Q8, R10, R11, R13, R17, R18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

Commit message: Small Gaggenau update
Parts:
- removed R29, R30: 47, Resistor_SMD:R_0603_1608Metric, symbol localparts:R_47_0603
- removed R32: 27, Resistor_SMD:R_1206_3216Metric, symbol Device:R
- added R29: 47, Resistor_SMD:R_1206_3216Metric, symbol Device:R
- Q10, Q11, Q12, Q13: value Q_PMOS -> 2301V
- R1: value 27 -> 47; LCSC C25367 -> C140015
Connections:
- net GND: now also Q7.3 (E), Q8.3 (E)
- net Kbraun: now also Q14.3 (D)
- net Krot: now also Q9.3 (D)
- net at R1.2: now also R29.1
- net at D7.2 (A2), R38.2: now also R29.2
- net at Q7.1 (C): now also R18.1; no longer Q8.1 (C)
- net at R17.1: now also Q8.1 (C); no longer Q8.3 (E)
Other:
- moved on the sheet: R17, R18, R36, R37
