File: breakout/fpc-03-15/fpc-03-15.kicad_sch (KiCad schematic)
At the start: 2 parts, among them J1 1-2328724-5, J2 Conn_01x16_Male

Commit message: A host of un-logged changes
Parts:
- J1: value 1-2328724-5 -> OLED FPC; symbol localstuff:FPC 15pin 0.3mm TE -> localstuff:OLED-96; LCSC C49166926 -> C49166942
Changed lines of the file:
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@@
 	)
 	(symbol
-		(lib_id "localstuff:FPC 15pin 0.3mm TE")
+		(lib_id "localstuff:OLED-96")
 		(at 40.64 41.91 0)
 		(unit 1)
@@
 		(fields_autoplaced yes)
 		(property "Reference" "J1"
-			(at 40.64 25.4 0)
+			(at 40.64 24.13 0)
 			(effects
 				(font
@@
 			)
 		)
-		(property "Value" "1-2328724-5"
-			(at 40.64 27.94 0)
+		(property "Value" "OLED FPC"
+			(at 40.64 26.67 0)
 			(effects
 				(font
@@
 		)
 		(property "Footprint" "localstuff:TE_1-2328724-5"
-			(at 40.64 41.91 0)
+			(at 29.21 62.23 0)
 			(effects
 				(font
@@
 			)
 		)
-		(property "Description" ""
-			(at 40.64 41.91 0)
+		(property "Description" "OLED 128x96, ForFuture Electron Tech"
+			(at 41.91 66.04 0)
 			(effects
 				(font
 					(size 1.27 1.27)
 				)
+				(hide yes)
 			)
 		)
 		(property "Comment" "1-2328724-5"
-			(at 40.64 41.91 0)
+			(at 34.29 64.77 0)
 			(effects
 				(font
@@
 			)
 		)
-		(property "LCSC" "C49166926"
+		(property "LCSC" "C49166942"
 			(at 40.64 41.91 0)
 			(effects
