File: wire/16/wire_16.kicad_pcb (KiCad board)
At the start: 2 copper layers, 18.8 x 20.4 mm, 3 parts, among them J1 Moat_Wire_16, J2 Moat_Wire_12

Commit message: A host of un-logged changes
Parts:
- removed the G*** at (36.0, 48.2)
- added G***: LOGO, localstuff:OSHW Logo 3mm Cu, F.Cu at (36.2, 46.6)
- added G***: LOGO, localstuff:OSHW Logo 3mm, F.Cu at (36.2, 46.6)
Connections:
- net Net-(J1-Pad1) renamed /KNX
- net Net-(J1-Pad2) renamed /GNDKNX
Routing:
- net /GNDPWR: track 36.0 -> 31.9 mm
- net /24V: track 33.5 -> 32.7 mm
- net /GND: vias 15 -> 14
Other:
- board text added: "V 2.3"
- board text removed: "V 2.2"
