File: wire/16/wire_16.kicad_sch (KiCad schematic)
At the start: 2 parts, among them J1 Moat_Wire_16, J2 Moat_Wire_12

Commit message: A host of un-logged changes
Connections:
- net KNX: now reaches J1.1 (KNX), J2.11 (KNX)
- net GNDKNX: now reaches J1.2 (GND_KNX), J2.12 (GND_KNX)
