File: wire/8/wire_8.kicad_pcb (KiCad board)
At the start: 2 copper layers, 18.8 x 13 mm, 2 parts, among them J1 Moat_Wire_8, J2 Moat_Wire_12

Commit message: A host of un-logged changes
Parts:
- added G***: LOGO, localstuff:OSHW Logo 2mm Cu, F.Cu at (35.3, 47.7)
- added G***: LOGO, localstuff:OSHW Logo 2mm, F.Cu at (35.3, 47.7)
Other:
- board text removed: "JLCJLCJLCJLC"
