File: base/heat_proc/heat_proc.kicad_pcb (KiCad board)
At the start: 4 copper layers, 41.2 x 32.7 mm, 64 parts, among them J1 USB_C_Receptacle, J10 Conn_01x02_Pin, J2 Moat_Heat_12, J3 Conn_01x01_Socket, J4 Conn_01x01_Socket, J5 Conn_01x01_Socket, J6 Conn_01x01_Socket, J7 Conn_01x01_Socket, J8 Conn_01x01_Socket, J9 1-2328724-5, Q1 HX2302A, Q13 HX2301V, Q2 HX2302A, Q3 HX2301V, Q4 HX2302A, Q5 HX2302A, Q6 HX2302A, Q7 HX2302A, U1 ESP32-S3-WROOM-2, U2 HX1001, U3 NS4168, U4 SD18OB261

Commit message: Slight moves
Parts:
- moved J8 4.07 mm to (135.7, 91.2)
- moved J7 3.99 mm to (124.7, 91.1)
- moved D1 1.45 mm to (134.9, 67.4)
- moved R12 1.25 mm to (124.7, 82.8)
- moved Prog1 0.37 mm to (117.0, 61.1)
Routing:
- net +5V: track 26.8 -> 11.3 mm
- net Net-(D1-A): track 23.9 -> 13.1 mm, vias 3 -> 1
- net /TPbottom: track 14.2 -> 18.5 mm
- net /Boot: track 31.9 -> 33.2 mm, vias 3 -> 2
- net /SCK: track 42.4 -> 41.2 mm
- net /Tleft: track 6.13 -> 6.72 mm
- net GND: track 100.6 -> 100.3 mm, vias 34 -> 35
Other:
- board size 41.2 x 32.7 mm -> 41.2 x 37.1 mm
